Commit message: fixed launch issue

File: custom_desc_moveit_pkg/urdf/ur_macro.xacro (robot description, xacro)
@@ -371,4 +371,26 @@
       <child link="${tf_prefix}tool0"/>
     </joint>
+    <link name="${tf_prefix}nozzle">
+      <visual>
+        <origin xyz="0 0 0" rpy="0 0 ${pi}"/>
+        <geometry>
+          <mesh filename="$(find custom_desc_moveit_pkg)/meshes/ur10e/collision/nozzle.stl" scale="1 1 1"/>
+        </geometry>
+      </visual>
+      <!--collision>
+        <origin xyz="0 0 0" rpy="0 0 ${pi}"/>
+        <geometry>
+          <mesh filename="$(find custom_desc_moveit_pkg)/meshes/ur10e/collision/nozzle.stl" scale="1 1 1"/>
+        </geometry>
+      </collision!-->
+      <xacro:cylinder_inertial radius="${base_inertia_radius}" length="${base_inertia_length}" mass="${base_mass}">
+        <origin xyz="0 0 0" rpy="0 0 0" />
+      </xacro:cylinder_inertial>
+    </link>
+    <joint name="${tf_prefix}tool0-nozzle" type="fixed">
+      <parent link="${tf_prefix}tool0"/>
+      <child link="${tf_prefix}nozzle"/>
+      <origin xyz="0 0 0" rpy="0 0 0"/>
+    </joint>
   </xacro:macro>
 </robot>

Commit message: testing proper packaging

File: custom_desc_moveit_pkg/urdf/ur_macro.xacro (robot description, xacro)
@@ -371,21 +371,4 @@
       <child link="${tf_prefix}tool0"/>
     </joint>
-    <link name="${tf_prefix}nozzle">
-      <visual>
-        <origin xyz="0 0 0" rpy="0 0 ${pi}"/>
-        <geometry>
-          <mesh filename="$(find custom_desc_moveit_pkg)/meshes/ur10e/collision/nozzle.stl" scale="1 1 1"/>
-        </geometry>
-      </visual>
-      <!--collision>
-        <origin xyz="0 0 0" rpy="0 0 ${pi}"/>
-        <geometry>
-          <mesh filename="$(find custom_desc_moveit_pkg)/meshes/ur10e/collision/nozzle.stl" scale="1 1 1"/>
-        </geometry>
-      </collision!-->
-      <xacro:cylinder_inertial radius="${base_inertia_radius}" length="${base_inertia_length}" mass="${base_mass}">
-        <origin xyz="0 0 0" rpy="0 0 0" />
-      </xacro:cylinder_inertial>
-    </link>
     <joint name="${tf_prefix}tool0-nozzle" type="fixed">
       <parent link="${tf_prefix}tool0"/>
@@ -393,4 +376,18 @@
       <origin xyz="0 0 0" rpy="0 0 0"/>
     </joint>
+    <link name="${tf_prefix}nozzle">
+      <visual>
+        <geometry>
+          <mesh filename="package://ur_custom_description/meshes/visual/nozzle.dae"/>
+        </geometry>
+        <origin rpy="0 0 0" xyz="0.75 0.5 -1"/>
+      </visual>
+      <collision>
+        <geometry>
+          <mesh filename="package://ur_custom_description/meshes/visual/nozzle.dae"/>
+        </geometry>
+        <origin rpy="0 0 0" xyz="0.75 0.5 -1"/>
+      </collision>
+    </link>
   </xacro:macro>
 </robot>
