Commit message: working moveit configuration (manually edit moveit_controllers.yaml)

File: ur_custom_control/urdf/ur_custom_controlled.urdf.xacro (robot description, xacro)
@@ -1,4 +1,4 @@
 <?xml version="1.0"?>
-<robot name="my_robot_cell" xmlns:xacro="http://ros.org/wiki/xacro">
+<robot name="custom_ur" xmlns:xacro="http://ros.org/wiki/xacro">
   <!--First, include the macro from our custom description-->
   <xacro:include filename="$(find ur_custom_description)/urdf/custom_ur_macro.xacro"/>
@@ -16,11 +16,12 @@
   <xacro:arg name="ur_output_recipe_filename" default="$(find ur_robot_driver)/resources/rtde_output_recipe.txt"/>
   <xacro:arg name="ur_input_recipe_filename" default="$(find ur_robot_driver)/resources/rtde_input_recipe.txt"/>
-  <xacro:arg name="use_mock_hardware" default="false" />
+  <xacro:arg name="use_mock_hardware" default="true" />
   <xacro:arg name="mock_sensor_commands" default="false" />
   <link name="world" />
   <!--Create the scene description including the robot-->
-  <xacro:my_robot_cell
+  <xacro:custom_ur
     parent="world"
     ur_type="$(arg ur_type)"
+    tf_prefix="$(arg ur_type)_"
     joint_limits_parameters_file="$(arg joint_limit_parameters_file)"
     kinematics_parameters_file="$(arg kinematics_parameters_file)"
@@ -29,5 +30,5 @@
   >
     <origin xyz="0 0 1" rpy="0 0 0" />
-  </xacro:my_robot_cell>
+  </xacro:custom_ur>
   <!--Create the control tag for the UR robot-->
   <xacro:ur_ros2_control

File: ur_custom_description/urdf/custom_ur_macro.xacro (robot description, xacro)
@@ -18,4 +18,16 @@
       <origin xyz="0.845 0.85 0" rpy="0 0 ${pi}" />
     </joint>
+    <!--This will create the specific robot-->
+    <xacro:ur_robot
+      name="${ur_type}"
+      tf_prefix="${ur_type}_"
+      parent="robot_mount"
+      joint_limits_parameters_file="${joint_limits_parameters_file}"
+      kinematics_parameters_file="${kinematics_parameters_file}"
+      physical_parameters_file="${physical_parameters_file}"
+      visual_parameters_file="${visual_parameters_file}"
+    >
+      <origin xyz="0 0 0" rpy="0 0 0" />
+    </xacro:ur_robot>
     <link name="${tf_prefix}nozzle">
       <visual>
@@ -35,18 +47,6 @@
       <parent link="${tf_prefix}tool0"/>
       <child link="${tf_prefix}nozzle"/>
-      <origin xyz="0 0 0" rpy="0 0 0"/>
+      <origin xyz="0 0 0" rpy="0 0 ${pi}"/>
     </joint>
-    <!--This will create the specific robot-->
-    <xacro:ur_robot
-      name="${ur_type}"
-      tf_prefix="${ur_type}_"
-      parent="robot_mount"
-      joint_limits_parameters_file="${joint_limits_parameters_file}"
-      kinematics_parameters_file="${kinematics_parameters_file}"
-      physical_parameters_file="${physical_parameters_file}"
-      visual_parameters_file="${visual_parameters_file}"
-    >
-      <origin xyz="0 0 0" rpy="0 0 0" />
-    </xacro:ur_robot>
   </xacro:macro>
 </robot>
