Commit message: cleaned up urdf

File: ur_custom_description/urdf/custom_ur.urdf.xacro (robot description, xacro)
@@ -2,5 +2,4 @@
 <robot name="custom_ur" xmlns:xacro="http://ros.org/wiki/xacro">
   <xacro:include filename="$(find ur_custom_description)/urdf/custom_ur_macro.xacro"/>
-  <xacro:arg name="tf_prefix" default="" />
   <xacro:arg name="ur_type" default="ur5"/>
   <xacro:arg name="joint_limits_parameters_file" default="$(find ur_description)/config/$(arg ur_type)/joint_limits.yaml"/>
@@ -12,5 +11,5 @@
   <xacro:custom_ur
     parent="world"
-    tf_prefix="$(arg tf_prefix)"
+    tf_prefix="$(arg ur_type)_"
     ur_type="$(arg ur_type)"
     joint_limits_parameters_file="$(arg joint_limits_parameters_file)"

File: ur_custom_description/urdf/custom_ur_macro.xacro (robot description, xacro)
@@ -1,5 +1,5 @@
 <?xml version="1.0"?>
 <robot xmlns:xacro="http://ros.org/wiki/xacro">
-  <xacro:include filename="$(find ur_custom_description)/urdf/ur_macro.xacro"/>
+  <xacro:include filename="$(find ur_description)/urdf/ur_macro.xacro"/>
   <xacro:macro name="custom_ur" params="
     tf_prefix
@@ -18,4 +18,23 @@
       <origin xyz="0.845 0.85 0" rpy="0 0 ${pi}" />
     </joint>
+    <link name="${tf_prefix}nozzle">
+      <visual>
+        <geometry>
+          <mesh filename="package://ur_custom_description/meshes/visual/nozzle_oriented.dae" scale= "0.9 0.9 0.9" />
+        </geometry>
+        <origin rpy="0 0 0" xyz="0 -0.018 0.15"/>
+      </visual>
+      <collision>
+        <geometry>
+          <mesh filename="package://ur_custom_description/meshes/visual/nozzle_oriented.dae" scale= "0.9 0.9 0.9"/>
+        </geometry>
+        <origin rpy="0 0 0" xyz="0 -0.018 0.15"/>
+      </collision>
+    </link>
+    <joint name="${tf_prefix}tool0-nozzle" type="fixed">
+      <parent link="${tf_prefix}tool0"/>
+      <child link="${tf_prefix}nozzle"/>
+      <origin xyz="0 0 0" rpy="0 0 0"/>
+    </joint>
     <!--This will create the specific robot-->
     <xacro:ur_robot

Commit message: moved robot model

File: ur_custom_description/urdf/custom_ur.urdf.xacro (robot description, xacro)
@@ -18,5 +18,5 @@
     visual_parameters_file="$(arg visual_parameters_file)"
     >
-      <origin xyz="0 0 1" rpy="0 0 0" />
+      <origin xyz="0 0 0" rpy="0 0 0" />
   </xacro:custom_ur>
 </robot>
