Commit message: description robot with welding nozzle

File: ur_custom_description/urdf/custom_ur_macro.xacro (robot description, xacro)
@@ -1,5 +1,5 @@
 <?xml version="1.0"?>
 <robot xmlns:xacro="http://ros.org/wiki/xacro">
-  <xacro:include filename="$(find ur_description)/urdf/ur_macro.xacro"/>
+  <xacro:include filename="$(find ur_custom_description)/urdf/ur_macro.xacro"/>
   <xacro:macro name="custom_ur" params="
     tf_prefix
@@ -30,40 +30,4 @@
       <origin xyz="0 0 0" rpy="0 0 0" />
     </xacro:ur_robot>
-    <joint name="${tf_prefix}tool0-nozzle" type="fixed">
-      <parent link="world"/>
-      <child link="${tf_prefix}table"/>
-      <origin xyz="0 0 0" rpy="0 0 0"/>
-    </joint>
-    <!--link name="${tf_prefix}nozzle">
-      <visual>
-        <geometry>
-          <mesh filename="$(find ur_custom_description)/meshes/fzi_table.dae"/>
-        </geometry>
-        <geometry>
-          <mesh filename="package://ur_custom_desciption/meshes/visual/fzi_table.dae"/>
-        </geometry>
-        <origin rpy="0 0 0" xyz="0.75 0.5 -1"/>
-      </visual>
-      <collision>
-        <geometry>
-          <mesh filename="$(find ur_custom_description)/meshes/fzi_table.dae"/>
-        </geometry>
-        <origin rpy="0 0 0" xyz="0.75 0.5 -1"/>
-      </collision>
-    </link!-->
-    <link name="${tf_prefix}table">
-      <visual>
-        <geometry>
-          <mesh filename="package://ur_custom_description/meshes/visual/nozzle.dae"/>
-        </geometry>
-        <origin rpy="0 0 0" xyz="0.75 0.5 -1"/>
-      </visual>
-      <collision>
-        <geometry>
-          <mesh filename="package://ur_custom_description/meshes/visual/nozzle.dae"/>
-        </geometry>
-        <origin rpy="0 0 0" xyz="0.75 0.5 -1"/>
-      </collision>
-    </link>
   </xacro:macro>
 </robot>

Commit message: moved robot position

File: ur_custom_description/urdf/custom_ur_macro.xacro (robot description, xacro)
@@ -16,5 +16,5 @@
       <parent link="world"/>
       <child link="robot_mount"/>
-      <origin xyz="0.845 0.85 0" rpy="0 0 ${pi}" />
+      <origin xyz="0 0 0" rpy="0 0 ${pi}" />
     </joint>
     <!--This will create the specific robot-->
@@ -47,5 +47,5 @@
       <parent link="${tf_prefix}tool0"/>
       <child link="${tf_prefix}nozzle"/>
-      <origin xyz="0 0 0" rpy="0 0 ${pi}"/>
+      <origin xyz="0 0 0.2" rpy="0 0 ${pi}"/>
     </joint>
   </xacro:macro>

Commit message: virtual tool endpoint

File: ur_custom_description/urdf/custom_ur_macro.xacro (robot description, xacro)
@@ -47,5 +47,11 @@
       <parent link="${tf_prefix}tool0"/>
       <child link="${tf_prefix}nozzle"/>
-      <origin xyz="0 0 0.2" rpy="0 0 ${pi}"/>
+      <origin xyz="0 0 0" rpy="0 0 ${pi}"/>
+    </joint>
+    <link name="tool_endpoint"/>
+    <joint name="${tf_prefix}tool0-tool_endpoint" type="fixed">
+      <parent link="${tf_prefix}tool0"/>
+      <child link="tool_endpoint"/>
+      <origin xyz="0 0.06 0.19" rpy="0 0 0"/>
     </joint>
   </xacro:macro>

Commit message: random fixes

File: ur_custom_description/urdf/custom_ur_macro.xacro (robot description, xacro)
@@ -16,5 +16,5 @@
       <parent link="world"/>
       <child link="robot_mount"/>
-      <origin xyz="0 0 0" rpy="0 0 ${pi}" />
+      <origin xyz="0 0 0" rpy="0 0 0" />
     </joint>
     <!--This will create the specific robot-->
