Commit message: test configs ur20

File: ur20_custom_description/urdf/custom_ur_macro_rotated.xacro (robot description, xacro)
@@ -16,5 +16,5 @@
       <parent link="world"/>
       <child link="robot_mount"/>
-      <origin xyz="0 0 0" rpy="0 0 ${pi}" />
+      <origin xyz="0 0 0" rpy="0 0 0" />
     </joint>
     <!--This will create the specific robot-->
@@ -28,5 +28,5 @@
       visual_parameters_file="${visual_parameters_file}"
     >
-      <origin xyz="0 0 0" rpy="0 0 0" />
+      <origin xyz="0 0 0" rpy="0 0 ${pi}" />
     </xacro:ur_robot>
     <link name="${tf_prefix}nozzle">
